File: EFR32MG22_module.brd (EAGLE design)
At the start: 16.8 x 23.1 mm, 35 parts, among them U1 EFR32MG22C224F512GN32, Y1 38.4MHZ, Y2 32.768KHz

Commit message: Add files via upload
Parts:
- moved C19 2.14 mm to (5.13, 15.6)
- moved E1 0.77 mm to (4.70, 17.1)
- moved TP1 0.77 mm to (4.70, 16.9)
- moved TP2 0.76 mm to (2.60, 16.9)
- moved Y2 0.51 mm to (14.0, 5.21)
- moved Y1 0.40 mm to (13.3, 10.5)
Routing:
- net GND: track 16.5 -> 18.2 mm, vias 144 -> 106
- net N$8: track 2.41 -> 1.34 mm
- net N$7: track 2.14 -> 2.97 mm
- net PC00: track 8.08 -> 8.83 mm, vias 1 -> 0
- net PC01: track 7.43 -> 7.80 mm, vias 1 -> 0
- net PC05: track 8.61 -> 8.83 mm, vias 1 -> 0
- net PC04: track 7.56 -> 7.72 mm, vias 1 -> 0
- net PC03: track 7.22 -> 7.21 mm, vias 1 -> 0
- net PC02: track 7.29 -> 7.30 mm, vias 1 -> 0
Other:
- board size 16.8 x 23.1 mm -> 16.8 x 22.3 mm
